Commit message: feat: 双目立体匹配 + 深度/点云节点 + 标定参数更新
- k7_camera 新增 stereo_depth 节点: 订阅 splitter 左右图 -> SGBM+WLS 视差 -> 深度图/视差/点云(PointCloud2 xyz+rgb)
- 离线脚本 generate_depth.py / stereo_match.py(SGBM+WLS+Q点云)
- 标定参数更新为新标定(fx=932, 基线21.9mm), 棋盘格物理5x7(内角点4x6, SB检测)
- launch stereo_depth.launch.py + 依赖 sensor_msgs_py/message_filters
- k7_description URDF 底盘尺寸调整
- .gitignore 忽略 *.png/*.csv 运行产物

File: ROS2_src/K7_ros2/src/k7_description/urdf/k7_robot.urdf (robot description, URDF)
Before this commit: robot k7_robot, 7 links, 6 joints
Links:
- link base_link: geometry visual box size=0.37 0.28 0.08
- link caster_link: geometry visual sphere radius=0.07
- link left_wheel_link: geometry visual cylinder length=0.04 radius=0.06
- link right_wheel_link: geometry visual cylinder length=0.04 radius=0.06
Joints:
- joint caster_joint: origin xyz=-0.13 0 -0.0325 rpy=0 0 0 -> xyz=0.085 0 -0.01 rpy=0 0 0
- joint left_wheel_joint: origin xyz=0 0.1645 -0.0625 rpy=0 0 0 -> xyz=-0.115 0.175 -0.02 rpy=0 0 0
- joint right_wheel_joint: origin xyz=0 -0.1645 -0.0625 rpy=0 0 0 -> xyz=-0.115 -0.175 -0.02 rpy=0 0 0
